File: hardware/MicroFans.sch (EAGLE design)
At the start: 29 parts, among them IC4 ATMEGA328P, IC7 OPA4251UA, J1 COMPUTER-PERIPHERAL-POWERVERT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, Y1 20Mhz

Commit message: Update board
Parts:
- added C3: 1uF, SparkFun-Capacitors:CAP0805
- added C7: 0.1uF, SparkFun-Passives:CAP1206
- added D1, D2: 3V6, SparkFun-DiscreteSemi:DIODE-ZENER-BZT52
- added IC1: (no value), SparkFun-PowerIC:V_REG_LM1117SOT223
- added JP7: (no value), SparkFun-Connectors:M03POLAR
- added R10: 47K, SparkFun-Passives:RESISTOR0805-RES
- added R11, R8: 8K6, SparkFun-Resistors:RESISTOR1206
- added R12, R9: 2K2, SparkFun-Resistors:RESISTOR1206
- added R13: 1K5, SparkFun-Passives:RESISTOR1206
- added R14, R15: 68, SparkFun-Passives:RESISTOR1206
- added R16: 220, SparkFun-Resistors:RESISTOR1206
- C1, C2: device SparkFun-Capacitors:CAPKIT -> SparkFun-Capacitors:CAP0805
- C4: value 0.1uF -> 1uF; device SparkFun-Capacitors:CAPKIT -> SparkFun-Capacitors:CAP0805
- C5, C6: device SparkFun-Capacitors:CAPKIT -> SparkFun-Passives:CAP1206
- JP1: value USB-A-S -> USB-A-SMD; device SparkFun-Connectors:USB-A-S -> SparkFun-Connectors:USB-A-SMD
- R1: device SparkFun-Resistors:RESISTOR1206 -> SparkFun-Passives:RESISTOR0805-RES
- R4: value 220 -> 47K; device SparkFun-Resistors:RESISTOR1206 -> SparkFun-Passives:RESISTOR0805-RES
- R6: value 47K -> 2K2
- R7: value 2K2 -> 47K; device SparkFun-Resistors:RESISTOR1206 -> SparkFun-Passives:RESISTOR0805-RES
- Y1: value 20Mhz -> 16MHZ
Connections:
- removed net +25V: IC5.IN
- removed net FAN1_TACH: JP5.3
- removed net FAN2_TACH: JP4.3
- removed net FAN3_TACH: JP3.3
- new net +12V: IC1.IN, IC3.IN, IC5.IN, IC6.IN, IC7P.V+, J1.12V
- new net N$1: IC1.OUT, JP7.2
- new net N$19: IC6.ADJ, IC7D.OUT, R8.1
- new net N$20: IC7D.-IN, R8.2, R9.1
- new net N$21: C3.1, IC7D.+IN, R7.1
- new net N$22: IC7C.-IN, R11.2, R12.1
- new net N$23: IC4.PC2(ADC2), R7.2
- new net N$24: C4.1, IC7C.+IN, R10.1
- new net N$25: IC1.ADJ, IC7C.OUT, R11.1
- new net N$26: D1.C, JP1.D-, R13.2, R15.1
- new net N$27: JP1.VBUS
- new net N$28: D2.C, JP1.D+, R14.1
- new net N$29: IC4.PD2(INT0), R14.2
- new net N$30: IC4.PD3(INT1), R15.2
- new net N$33: J1.5V, R16.2
- new net N$34: IC4.PC3(ADC3), R10.2
- new net SENSE1: IC4.PB0(ICP), JP5.3
- new net SENSE2: IC4.PB1(OC1A), JP4.3
- new net SENSE3: IC4.PB2(SS/OC1B), JP3.3
- new net SENSE4: IC4.PD7(AIN1), JP7.3
- net +5V: now also C7.1, R13.1; no longer C4.1, J1.5V, R4.2
- net GND: now also C1.2, C2.2, C3.2, C7.2, D1.A, D2.A, IC7P.V-, JP1.GND, JP7.1, R12.2, R6.2, R9.2; no longer R7.2
- net N$12: now also IC4.PC1(ADC1), R4.2; no longer R6.2
- net N$13: now also IC6.OUT, JP3.2; no longer JP4.2
- net N$15: now also C1.1; no longer C2.1
- net N$16: now also R3.1; no longer C2.2, R7.1
- net N$17: now also C2.1, R4.1; no longer C1.1, R6.1
- net N$18: now also R6.1; no longer C1.2, R3.1
- net N$5: now also IC4.PC0(ADC0)
- net N$7: now also R16.1; no longer R4.1
- net N$8: now also IC5.OUT, JP4.2; no longer JP3.2
Other:
- moved on the sheet: C1, C2, C4, C5, C6, IC4, IC6, IC7C, IC7D, ICSP, J1, JP3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

Commit message: More work on board
Parts:
- removed IC7: OPA4251UA, linear:OPA4251UA
- added IC2: (no value), SparkFun-PowerIC:V_REG_LM1117SOT223
- added R17, R18, R19, R20: 10K, SparkFun-Resistors:RESISTOR0805-RES
- C5, C6: device SparkFun-Passives:CAP1206 -> SparkFun-Capacitors:CAP0805
- IC4: value ATMEGA328P -> (none); device SparkFun-DigitalIC:ATMEGA328_SMT -> SparkFun-PowerIC:V_REG_LM1117SOT223
- IC5: value (none) -> ATMEGA328P; device SparkFun-PowerIC:V_REG_LM1117SOT223 -> SparkFun-DigitalIC:ATMEGA328_SMT
- IC6: value (none) -> OPA4251UA; device SparkFun-PowerIC:V_REG_LM1117SOT223 -> linear:OPA4251UA
- R1, R10, R4, R7: device SparkFun-Passives:RESISTOR0805-RES -> SparkFun-Resistors:RESISTOR0805-RES
- R11, R12, R16, R2, R3, R5, R6, R8, R9: device SparkFun-Resistors:RESISTOR1206 -> SparkFun-Resistors:RESISTOR0805-RES
- R13, R14, R15: device SparkFun-Passives:RESISTOR1206 -> SparkFun-Resistors:RESISTOR0805-RES
Connections:
- net N$26 renamed D-
- net N$28 renamed D+
- removed net N$4: ICSP.5
- net +12V: now also IC2.IN, IC4.IN, IC6P.V+; no longer IC5.IN, IC6.IN, IC7P.V+
- net +5V: now also IC5.AVCC, IC5.VCC@1, IC5.VCC@2, R17.1, R18.1, R19.1, R20.1; no longer IC4.AVCC, IC4.VCC@1, IC4.VCC@2
- net GND: now also IC5.AGND, IC5.GND@1, IC5.GND@2, IC6P.V-; no longer IC4.AGND, IC4.GND@1, IC4.GND@2, IC7P.V-
- net N$10: now also IC5.PB5(SCK)
- net N$11: now also IC5.PB3(MOSI/OC2)
- net N$12: now also IC5.PC1(ADC1); no longer IC4.PC1(ADC1)
- net N$13: now also IC2.OUT; no longer IC6.OUT
- net N$14: now also IC3.ADJ, IC6B.OUT; no longer IC5.ADJ, IC7B.OUT
- net N$15: now also IC6A.+IN; no longer IC7A.+IN
- net N$16: now also IC6A.-IN; no longer IC7A.-IN
- net N$17: now also IC6B.+IN; no longer IC7B.+IN
- net N$18: now also IC6B.-IN; no longer IC7B.-IN
- net N$19: now also IC2.ADJ, IC6D.OUT; no longer IC6.ADJ, IC7D.OUT
- net N$2: now also IC4.ADJ, IC6A.OUT; no longer IC3.ADJ, IC7A.OUT
- net N$20: now also IC6D.-IN; no longer IC7D.-IN
- net N$21: now also IC6D.+IN; no longer IC7D.+IN
- net N$22: now also IC6C.-IN; no longer IC7C.-IN
- net N$23: now also IC5.PC2(ADC2); no longer IC4.PC2(ADC2)
- net N$24: now also IC6C.+IN; no longer IC7C.+IN
- net N$25: now also IC6C.OUT; no longer IC7C.OUT
- net N$29: now also IC5.PD2(INT0); no longer IC4.PD2(INT0)
- net N$3: now also IC5.PB4(MISO)
- net N$30: now also IC5.PD3(INT1); no longer IC4.PD3(INT1)
- net N$31: now also IC4.OUT; no longer IC3.OUT
- net N$34: now also IC5.PC3(ADC3); no longer IC4.PC3(ADC3)
- net N$5: now also IC5.PC0(ADC0); no longer IC4.PC0(ADC0)
- net N$6: now also IC5.PB6(XTAL1/TOSC1); no longer IC4.PB6(XTAL1/TOSC1)
- net N$8: now also IC3.OUT; no longer IC5.OUT
- net N$9: now also IC5.PB7(XTAL2/TOSC2); no longer IC4.PB7(XTAL2/TOSC2)
- net RESET: now also IC5.PC6(/RESET), ICSP.5; no longer IC4.PC6(/RESET)
- net SENSE1: now also IC5.PB0(ICP), R17.2; no longer IC4.PB0(ICP)
- net SENSE2: now also IC5.PB1(OC1A), R18.2; no longer IC4.PB1(OC1A)
- net SENSE3: now also IC5.PB2(SS/OC1B), R19.2; no longer IC4.PB2(SS/OC1B)
- net SENSE4: now also IC5.PD7(AIN1), R20.2; no longer IC4.PD7(AIN1)
Other:
- moved on the sheet: IC3, ICSP, JP3, JP4, JP5, JP7

Commit message: Updated board with LM2341
Parts:
- removed C4: 1uF, SparkFun-Capacitors:CAP0805
- removed IC2: (no value), SparkFun-PowerIC:V_REG_LM1117SOT223
- removed IC6: OPA4251UA, linear:OPA4251UA
- removed JP7: (no value), SparkFun-Connectors:M03POLAR
- removed R17, R18, R19, R20: 10K, SparkFun-Resistors:RESISTOR0805-RES
- removed R8: 8K6, SparkFun-Resistors:RESISTOR0805-RES
- added HOLE3: STAND-OFF, SparkFun:STAND-OFF
- added USB: USB-A-SMD, SparkFun-Connectors:USB-A-SMD
- C3: value 1uF -> 0.1uF
- C7: device SparkFun-Passives:CAP1206 -> SparkFun-Capacitors:CAP0805
- IC1: value (none) -> OPA2251UA; device SparkFun-PowerIC:V_REG_LM1117SOT223 -> linear:OPA2251UA
- IC3, IC4: value (none) -> LM2941TO220-V; device SparkFun-PowerIC:V_REG_LM1117SOT223 -> lm2941:LM2941TO220-V
- JP1: value USB-A-SMD -> (none); device SparkFun-Connectors:USB-A-SMD -> SparkFun-Connectors:M03POLAR
- JP2: value STAND-OFF -> (none); device SparkFun:STAND-OFF -> SparkFun-Connectors:M03POLAR
- JP5: device SparkFun-Connectors:M03POLAR -> SparkFun-Connectors:M02PTH
- R10, R7: value 47K -> 10K
- R11: value 8K6 -> 10K
- R12, R9: value 2K2 -> 10K
- renumbered JP6 to HOLE2, JP8 to HOLE4, JP9 to HOLE1
Connections:
- removed net N$19: IC2.ADJ, IC6D.OUT, R8.1
- removed net N$20: IC6D.-IN, R8.2, R9.1
- removed net N$21: C3.1, IC6D.+IN, R7.1
- removed net N$22: IC6C.-IN, R11.2, R12.1
- removed net N$23: IC5.PC2(ADC2), R7.2
- removed net N$24: C4.1, IC6C.+IN, R10.1
- removed net N$25: IC1.ADJ, IC6C.OUT, R11.1
- removed net N$27: JP1.VBUS
- removed net N$31: IC4.OUT, JP5.2
- removed net N$33: J1.5V, R16.2
- removed net N$34: IC5.PC3(ADC3), R10.2
- new net N$4: IC5.PD1(TXD), JP5.2
- net +12V: now also IC1A.V+; no longer IC1.IN, IC2.IN, IC6P.V+
- net +5V: now also J1.5V, R10.1, R11.1, R12.1, R16.2, R7.1, R9.1; no longer R17.1, R18.1, R19.1, R20.1
- net D+: now also USB.D+; no longer JP1.D+
- net D-: now also USB.D-; no longer JP1.D-
- net GND: now also IC1A.V-, IC3.GND, IC3.ON, IC4.GND, IC4.ON, JP1.1, JP2.1, USB.GND; no longer C4.2, IC6P.V-, JP1.GND, JP5.1, JP7.1, R12.2, R9.2
- net N$1: now also IC5.PD0(RXD), JP5.1; no longer IC1.OUT, JP7.2
- net N$13: now also IC4.OUT, JP4.2; no longer IC2.OUT
- net N$14: now also IC1B.OUT, IC4.ADJ; no longer IC3.ADJ, IC6B.OUT
- net N$15: now also IC1A.+IN; no longer IC6A.+IN
- net N$16: now also IC1A.-IN; no longer IC6A.-IN
- net N$17: now also IC1B.+IN; no longer IC6B.+IN
- net N$18: now also IC1B.-IN; no longer IC6B.-IN
- net N$2: now also IC1A.OUT, IC3.ADJ; no longer IC4.ADJ, IC6A.OUT
- net N$8: now also JP1.2, JP2.2; no longer JP4.2
- net RESET: now also C3.1, R7.2
- net SENSE1: now also IC5.PC2(ADC2), JP1.3, R9.2; no longer IC5.PB0(ICP), JP5.3, R17.2
- net SENSE2: now also IC5.PC3(ADC3), JP2.3, R10.2; no longer IC5.PB1(OC1A), JP4.3, R18.2
- net SENSE3: now also IC5.PB1(OC1A), R11.2; no longer IC5.PB2(SS/OC1B), R19.2
- net SENSE4: now also IC5.PB2(SS/OC1B), JP4.3, R12.2; no longer IC5.PD7(AIN1), JP7.3, R20.2
Other:
- moved on the sheet: C2, C3, J1, JP3, JP4, R10, R11, R12, R4, R5, R6, R7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
