File: hardware/MicroBreeze.brd (EAGLE design)
At the start: 52.1 x 38.1 mm, 41 parts, among them IC1 OPA2251UA, IC3 LM2941TO220-V, IC4 LM2941TO220-V, IC5 ATMEGA328P, Y1 16MHZ

Commit message: Add filter caps
Parts:
- added C4, C8: 22uF, SparkFun-Capacitors:1210
- moved R16 42.4 mm to (12.1, 2.86), turned to 180 degrees
- moved PWR 42.0 mm to (17.8, 1.91), turned to 0 degrees
Connections:
- net GND: now also C4.2, C8.2
- net N$13: now also C8.1
- net N$8: now also C4.1
Routing:
- net +5V: track 92.9 -> 113.1 mm, vias 4 -> 6
- net GND: track 68.1 -> 80.7 mm
- net N$13: track 29.2 -> 40.0 mm, vias 0 -> 1
- net N$8: track 20.7 -> 27.0 mm
- net N$7: track 3.01 -> 3.71 mm

Commit message: Board updates
Parts:
- added R17, R8: 240, SparkFun-Resistors:0805
- C4, C8: value 22uF -> 47uF; device SparkFun-Capacitors:1210 -> SparkFun-Capacitors:EIA3528
- moved C1 0.64 mm to (26.7, 24.8)
- moved C8 0.64 mm to (43.2, 3.81), turned to 270 degrees
- turned C4 to 270 degrees
Connections:
- removed net N$14: IC1.7, IC4.1, R5.1
- new net N$19: IC1.7, IC4.1, R5.1, R8.1
- net GND: now also C4.C, C8.C; no longer C4.2, C8.2
- net N$13: now also C8.A, R8.2; no longer C8.1
- net N$2: now also R17.1
- net N$8: now also C4.A, R17.2; no longer C4.1
Routing:
- net N$19: track 0.00 -> 20.3 mm, vias 0 -> 1
- net N$14: track 20.2 -> 0.00 mm, vias 1 -> 0
- net N$8: track 27.0 -> 46.7 mm
- net +5V: track 113.1 -> 108.6 mm
- net N$2: track 16.8 -> 19.0 mm, vias 0 -> 1
- net N$13: track 40.0 -> 41.1 mm, vias 1 -> 0
- net N$10: track 20.9 -> 22.0 mm
- net GND: track 80.7 -> 79.9 mm
